Commit message: Add foot inertia.

File: resources/robots/cyberdog2/urdf/cyberdog2.urdf (robot description, URDF)
Before this commit: robot cyberdog2_description, 19 links, 18 joints
Links:
- link FL_foot: mass None -> 0.25
- link FR_foot: mass None -> 0.25
- link RL_foot: mass None -> 0.25
- link RR_foot: mass None -> 0.25
