Commit message: Update urdf dir.

File: resources/robots/go2/urdf/go2.urdf (robot description, URDF)
Before this commit: robot go2_description, 29 links, 28 joints
Links:
- link FL_calf: geometry collision cylinder length=0.12 radius=0.012; visual mesh filename=/home/yuchen/usetest/RL/legged_gym/resources/robots/go2/mes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
- link FL_foot: geometry collision sphere radius=0.022; visual mesh filename=/home/yuchen/usetest/RL/legged_gym/resources/robots/go2/mes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
- link FL_hip: geometry collision cylinder length=0.04 radius=0.046; visual mesh filename=/home/yuchen/usetest/RL/legged_gym/resources/robots/go2/mes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
- link FL_thigh: geometry collision box size=0.11 0.0245 0.034; visual mesh filename=/home/yuchen/usetest/RL/legged_gym/resources/robots/go2/mes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
- link FR_calf: geometry collision cylinder length=0.12 radius=0.013; visual mesh filename=/home/yuchen/usetest/RL/legged_gym/resources/robots/go2/mes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
- link FR_foot: geometry collision sphere radius=0.022; visual mesh filename=/home/yuchen/usetest/RL/legged_gym/resources/robots/go2/mes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
- link FR_hip: geometry collision cylinder length=0.04 radius=0.046; visual mesh filename=/home/yuchen/usetest/RL/legged_gym/resources/robots/go2/mes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
- link FR_thigh: geometry collision box size=0.11 0.0245 0.034; visual mesh filename=/home/yuchen/usetest/RL/legged_gym/resources/robots/go2/mes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
- link RL_calf: geometry collision cylinder length=0.12 radius=0.013; visual mesh filename=/home/yuchen/usetest/RL/legged_gym/resources/robots/go2/mes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
- link RL_foot: geometry collision sphere radius=0.022; visual mesh filename=/home/yuchen/usetest/RL/legged_gym/resources/robots/go2/mes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
- link RL_hip: geometry collision cylinder length=0.04 radius=0.046; visual mesh filename=/home/yuchen/usetest/RL/legged_gym/resources/robots/go2/mes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
- link RL_thigh: geometry collision box size=0.11 0.0245 0.034; visual mesh filename=/home/yuchen/usetest/RL/legged_gym/resources/robots/go2/mes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
- link RR_calf: geometry collision cylinder length=0.12 radius=0.013; visual mesh filename=/home/yuchen/usetest/RL/legged_gym/resources/robots/go2/mes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
- link RR_foot: geometry collision sphere radius=0.022; visual mesh filename=/home/yuchen/usetest/RL/legged_gym/resources/robots/go2/mes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
- link RR_hip: geometry collision cylinder length=0.04 radius=0.046; visual mesh filename=/home/yuchen/usetest/RL/legged_gym/resources/robots/go2/mes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
- link RR_thigh: geometry collision box size=0.11 0.0245 0.034; visual mesh filename=/home/yuchen/usetest/RL/legged_gym/resources/robots/go2/mes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
- link base: geometry collision box size=0.3762 0.0935 0.114; visual mesh filename=/home/yuchen/usetest/RL/legged_gym/resources/robots/go2/mes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
